File: hardware/AUV-HydroMap-6D-System/AUV-HydroMap-6D-System.kicad_sch (KiCad schematic)
At the start: 0 parts

Commit message: hw: started the implementation of the STM32WB55CEUx
Parts:
- added C1, C8: 4.7uF, symbol Device:C_Small
- added C10, C12, C2, C3, C4, C5, C9: 100nF, symbol Device:C_Small
- added C11: 100pF, symbol Device:C_Small
- added C6: 1.0uF, symbol Device:C_Small
- added C7: 10nF, symbol Device:C_Small
- added U1: STM32WB55CEUx, Package_DFN_QFN:QFN-48-1EP_7x7mm_P0.5mm_EP5.6x5.6mm, symbol MCU_ST_STM32WB:STM32WB55CEUx
Connections:
- new net +3V3: C1.1, C10.1, C11.1, C2.1, C3.1, C4.1, C5.1, C6.1, C7.1, C8.1, C9.1, U1.1 (VBAT), U1.20 (VDD), U1.23 (VDDRF), U1.34 (VDDSMPS), U1.35 (VDD), U1.48 (VDD), U1.8 (VDDA)
- new net GND: C1.2, C10.2, C11.2, C12.2, C2.2, C3.2, C4.2, C5.2, C6.2, C7.2, C8.2, C9.2, U1.22 (VSSRF), U1.32 (VSSSMPS), U1.49 (VSS)
- new net VBUS: C12.1, U1.40 (VDDUSB)
- no-connect marks 0 -> 26
Other:
- note added: "Decoupling capacitor VBAT/VDD"
- note added: "Decoupling capacitor VDDA"
- note added: "Decoupling capacitor VDDRF"
- note added: "Decoupling capacitor VDDSMPS"
- note added: "Decoupling capacitor VDDUSB"
